File: 43 x 43 KiCad Design 2/ta-expt-v2.kicad_sch (KiCad schematic)
At the start: 47 parts, among them IC1 BAR43SFILM, IC2 STS5PF30L, IC3 STM32L496VGT3, IC4 IS25LP128F-JBLA3, J1 Conn_01x05, J2 Conn_01x04, J3 USB_C_Receptacle_USB2.0, J4 Conn_01x05, J5 4-174639-8, J6 Conn_01x04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

Commit message: Updated 43 x 43 mm Design 2 with QUAD SPI BK 2 NCS. NEED TO BE CHANGED ON DESIGN 1 AS WELL. PCB NEEDS TO BE UPDATED ON BOTH OF THEM.
Connections:
- net QUADSPI_BK2_NCS: now reaches IC3.84 (PD3)
- net QUADSPI_BK2_NCS: now also IC4.1 (CE#), R7.2
- removed net QUADSPI_BK1_NCS: IC3.25 (PA2), IC4.1 (CE#), R7.2
Changed lines of the file:
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@@
+		)
+	)
+	(label "QUADSPI_BK2_NCS"
+		(at 241.3 92.71 90)
+		(fields_autoplaced yes)
+		(effects
+			(font
+				(size 1.27 1.27)
+			)
+			(justify left bottom)
 		)
 	)
@@
 		)
 	)
-	(label "QUADSPI_BK1_NCS"
-		(at 193.04 176.53 180)
-		(fields_autoplaced yes)
-		(effects
-			(font
-				(size 1.27 1.27)
-			)
-			(justify right bottom)
-		)
-	)
 	(label "VDD_FILT"
 		(at 185.42 107.95 0)
@@
 		)
 	)
-	(label "QUADSPI_BK1_NCS"
+	(label "QUADSPI_BK2_NCS"
 		(at 279.4 40.64 180)
 		(fields_autoplaced yes)
